File: device/statuspanel.sch (EAGLE design)
At the start: 8 parts

Commit message: feat(device): Add a reset button to the custom PCB (#379)
This also includes drive-by changes to use SMD resistors, and correct the resistance of the status LED resistor.
Parts:
- added RESET: (no value), switch-omron:10-XX
- R1: value 5.1 -> 330; device adafruit:R-US_0411/12 -> adafruit:R-US_R0805
- R2, R3: device adafruit:R-US_0411/12 -> adafruit:R-US_R0805
- renumbered STAT. to STATUS
Connections:
- new net RST: HUZZAH32.RST, RESET.S
- net GND: now also RESET.P
Changed lines of the file:
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@@
 <layers>
 <layer number="1" name="Top" color="4" fill="1" visible="no" active="no"/>
-<layer number="2" name="Route2" color="1" fill="3" visible="no" active="no"/>
+<layer number="2" name="Route2" color="16" fill="1" visible="no" active="no"/>
 <layer number="3" name="Route3" color="4" fill="3" visible="no" active="no"/>
 <layer number="4" name="Route4" color="1" fill="4" visible="no" active="no"/>
@@
 <layer number="13" name="Route13" color="4" fill="5" visible="no" active="no"/>
 <layer number="14" name="Route14" color="1" fill="6" visible="no" active="no"/>
-<layer number="15" name="Route15" color="4" fill="6" visible="no" active="no"/>
+<layer number="15" name="Route15" color="23" fill="1" visible="no" active="no"/>
 <layer number="16" name="Bottom" color="1" fill="1" visible="no" active="no"/>
 <layer number="17" name="Pads" color="2" fill="1" visible="no" active="no"/>
 <layer number="18" name="Vias" color="2" fill="1" visible="no" active="no"/>
 <layer number="19" name="Unrouted" color="6" fill="1" visible="no" active="no"/>
-<layer number="20" name="Dimension" color="15" fill="1" visible="no" active="no"/>
-<layer number="21" name="tPlace" color="14" fill="1" visible="no" active="no"/>
+<layer number="20" name="Dimension" color="24" fill="1" visible="no" active="no"/>
+<layer number="21" name="tPlace" color="7" fill="1" visible="no" active="no"/>
 <layer number="22" name="bPlace" color="7" fill="1" visible="no" active="no"/>
 <layer number="23" name="tOrigins" color="15" fill="1" visible="no" active="no"/>
@@
 <part name="AUTO" library="adafruit" library_urn="urn:adsk.eagle:library:420" deviceset="EG1218" device="S" package3d_urn="urn:adsk.eagle:package:6240649/1"/>
 <part name="UNPAIR" library="switch-omron" library_urn="urn:adsk.eagle:library:377" deviceset="10-XX" device="" package3d_urn="urn:adsk.eagle:package:27496/1"/>
-<part name="STAT." library="adafruit" library_urn="urn:adsk.eagle:library:420" deviceset="LED" device="3MM" package3d_urn="urn:adsk.eagle:package:6240537/1"/>
-<part name="R1" library="adafruit" library_urn="urn:adsk.eagle:library:420" deviceset="R-US_" device="0411/12" package3d_urn="urn:adsk.eagle:package:6240605/1" value="5.1"/>
-<part name="R2" library="adafruit" library_urn="urn:adsk.eagle:library:420" deviceset="R-US_" device="0411/12" package3d_urn="urn:adsk.eagle:package:6240605/1" value="4.7K"/>
-<part name="R3" library="adafruit" library_urn="urn:adsk.eagle:library:420" deviceset="R-US_" device="0411/12" package3d_urn="urn:adsk.eagle:package:6240605/1" value="4.7K"/>
+<part name="STATUS" library="adafruit" library_urn="urn:adsk.eagle:library:420" deviceset="LED" device="3MM" package3d_urn="urn:adsk.eagle:package:6240537/1"/>
+<part name="R1" library="adafruit" library_urn="urn:adsk.eagle:library:420" deviceset="R-US_" device="R0805" package3d_urn="urn:adsk.eagle:package:6240566/1" value="330"/>
+<part name="R2" library="adafruit" library_urn="urn:adsk.eagle:library:420" deviceset="R-US_" device="R0805" package3d_urn="urn:adsk.eagle:package:6240566/1" value="4.7K"/>
+<part name="R3" library="adafruit" library_urn="urn:adsk.eagle:library:420" deviceset="R-US_" device="R0805" package3d_urn="urn:adsk.eagle:package:6240566/1" value="4.7K"/>
+<part name="RESET" library="switch-omron" library_urn="urn:adsk.eagle:library:377" deviceset="10-XX" device="" package3d_urn="urn:adsk.eagle:package:27496/1"/>
 </parts>
 <sheets>
@@
 <attribute name="VALUE" x="65.405" y="16.51" size="1.778" layer="96" rot="R180"/>
 </instance>
-<instance part="STAT." gate="G$1" x="119.38" y="30.48" smashed="yes" rot="R270">
+<instance part="STATUS" gate="G$1" x="119.38" y="30.48" smashed="yes" rot="R270">
 <attribute name="NAME" x="114.808" y="24.384" size="1.778" layer="95"/>
 <attribute name="VALUE" x="114.808" y="24.765" size="1.778" layer="96"/>
@@
 <attribute name="NAME" x="102.87" y="16.7386" size="1.778" layer="95"/>
 <attribute name="VALUE" x="102.87" y="11.938" size="1.778" layer="96"/>
+</instance>
+<instance part="RESET" gate="1" x="68.58" y="0" smashed="yes" rot="R90">
+<attribute name="NAME" x="71.12" y="-6.35" size="1.778" layer="95" rot="R180"/>
+<attribute name="VALUE" x="65.405" y="-3.81" size="1.778" layer="96" rot="R180"/>
 </instance>
 </instances>
@@
 <wire x1="55.88" y1="86.36" x2="55.88" y2="68.58" width="0.1524" layer="91"/>
 </segment>
+<segment>
+<pinref part="RESET" gate="1" pin="P"/>
+<wire x1="73.66" y1="0" x2="76.2" y2="0" width="0.1524" layer="91"/>
+<label x="76.2" y="0" size="0.8128" layer="95" xref="yes"/>
+</segment>
 </net>
 <net name="AUTO" class="0">
@@
 <net name="STATUS" class="0">
 <segment>
-<pinref part="STAT." gate="G$1" pin="A"/>
+<pinref part="STATUS" gate="G$1" pin="A"/>
 <wire x1="121.92" y1="30.48" x2="124.46" y2="30.48" width="0.1524" layer="91"/>
 <label x="124.46" y="30.48" size="0.8128" layer="95" xref="yes"/>
@@
 <net name="N$3" class="0">
 <segment>
-<pinref part="STAT." gate="G$1" pin="C"/>
+<pinref part="STATUS" gate="G$1" pin="C"/>
 <wire x1="114.3" y1="30.48" x2="111.76" y2="30.48" width="0.1524" layer="91"/>
 <pinref part="R1" gate="G$1" pin="2"/>
@@
 </segment>
 </net>
+<net name="RST" class="0">
+<segment>
+<pinref part="HUZZAH32" gate="G$1" pin="RST"/>
+<wire x1="134.62" y1="48.26" x2="139.7" y2="48.26" width="0.1524" layer="91"/>
+<label x="139.7" y="48.26" size="0.8128" layer="95" xref="yes"/>
+</segment>
+<segment>
+<pinref part="RESET" gate="1" pin="S"/>
+<wire x1="63.5" y1="0" x2="60.96" y2="0" width="0.1524" layer="91"/>
+<label x="60.96" y="0" size="0.8128" layer="95" rot="R180" xref="yes"/>
+</segment>
+</net>
